File: PCB/plai.kicad_sch (KiCad schematic)
At the start: 22 parts, among them SW1 SW_Push, SW10 RotaryEncoder_Switch, SW2 SW_Push, SW3 SW_Push, SW4 SW_Push, SW5 SW_Push, SW6 SW_Push, SW7 SW_Push, SW8 SW_Push, SW9 SW_Push, U1 ER_OLEDM0.91_1x-I2C, U2 MOUDLE-SEEEDUINO-XIAO

Commit message: Fullyt Routed PCB Beautifully Routed + Some additions ot the firmware
Connections:
- net ROW3 is gone; now on net ROW2: U2.8 (PB09_A7_D7_RX)
- net COL0: now also U2.1 (PA02_A0_D0)
- net COL1: now also U2.2 (PA4_A1_D1); no longer U2.1 (PA02_A0_D0)
- net COL2: now also U2.3 (PA10_A2_D2); no longer U2.2 (PA4_A1_D1)
- net COL3: now also U2.4 (PA11_A3_D3); no longer U2.3 (PA10_A2_D2)
- net ROW0: now also U2.7 (PB08_A6_D6_TX)
- net ROW1: now also U2.11 (PA6_A10_D10_MOSI); no longer U2.4 (PA11_A3_D3)
- net ROW2: no longer U2.7 (PB08_A6_D6_TX)
